File: KiCad/USB-2-232.kicad_pcb (KiCad board)
At the start: 2 copper layers, 79.7 x 35.1 mm, 29 parts, among them J1 Conn_01x06_Male, J2 Conn_01x02_Male, J3 Conn_01x05_Male, SW1 SW_DIP_x06, SW2 SW_MEC_5E, U1 MAX232, U2 PICO_RP2040

Commit message: PCBv2
Fixed the silkscreen for J1 and fixed the crossed traces on serial connector.
Moved some traces around to make it look nicer and changed the PFP logo so hopefully JLC can't feck it up.
Parts:
- G***: footprint USB-2-232:pfp-1050-flip -> USB-2-232:pfp-1050-v2
- J1: footprint usbpico:PinHeader_ALT_SERIAL_OUT -> USB-2-232:PinHeader_ALT_SERIAL_OUT
- J2: value Conn_01x02_Male -> PWR-PINH
- J3: value Conn_01x05_Male -> USB-PINHEADER
- rs232_1: footprint Connector_Dsub:DSUB-9_Male_Horizontal_P2.77x2.84mm_EdgePinOffset7.70mm_Housed_MountingHolesOffset9.12mm -> Connector_Dsub:DSUB-9_Female_Horizontal_P2.77x2.84mm_EdgePinOffset7.70mm_Housed_MountingHolesOffset9.12mm
- moved rs232_1 11.1 mm to (131.6, 98.7)
Connections:
- net Net-(JP1-Pad3) renamed +3V3
- J1 pad 1: GND -> Net-(J1-Pad1)
- J1 pad 5: Net-(J1-Pad5) -> GND
- U1 pad 14: Net-(J1-Pad5) -> Net-(J1-Pad2)
- U1 pad 7: Net-(J1-Pad3) -> Net-(J1-Pad1)
- U1 pad 8: Net-(J1-Pad2) -> Net-(J1-Pad3)
- rs232_1 pad 2: Net-(J1-Pad4) -> Net-(J1-Pad2)
- rs232_1 pad 3: Net-(J1-Pad5) -> Net-(J1-Pad4)
- rs232_1 pad 7: Net-(J1-Pad2) -> Net-(J1-Pad3)
- rs232_1 pad 8: Net-(J1-Pad3) -> Net-(J1-Pad1)
Routing:
- net Net-(J1-Pad1): track 0.00 -> 56.4 mm, vias 0 -> 1
- net Net-(J1-Pad5): track 46.4 -> 0.00 mm
- net Net-(J1-Pad2): track 71.4 -> 49.1 mm, vias 1 -> 0
- net Net-(J1-Pad3): track 73.0 -> 58.9 mm
- net Net-(J1-Pad4): track 51.6 -> 45.3 mm, vias 0 -> 2
- net Net-(SW1-Pad4): track 25.7 -> 23.7 mm
- net Net-(U1-Pad11): track 17.8 -> 18.5 mm
- net Net-(R3-Pad2): track 20.6 -> 20.1 mm
- net +5V: track 81.3 -> 81.8 mm, vias 3 -> 2
- net GND: vias 4 -> 2
