File: KiCad/Slim/USB-2-232-slim.kicad_pcb (KiCad board)
At the start: 2 copper layers, 66.5 x 32 mm, 26 parts, among them J2 PWR-PINH, SW2 RESET, U1 MAX232, U2 PICO_RP2040

Commit message: Fixed misplaced silkscreen
Parts:
- moved G*** 2.24 mm to (155.2, 97.6)
